Commit message: working_RDS

File: urdf/delta.urdf (robot description, URDF)
Before this commit: robot delta, 29 links, 28 joints
Links:
- link base_link: geometry collision cylinder length=0.0127 radius=0.111; visual cylinder length=0.0127 radius=0.111
- link end_link: geometry collision cylinder length=0.00635 radius=0.05; visual cylinder length=0.00635 radius=0.05
Joints:
- joint front_delta_arm_joint: limit lower=-1.0471975511965976 upper=1.0471975511965976 effort=6 velocity=8 -> lower=-0.3490658503988659 upper=1.5707963267948966 effort=6 velocity=8; origin xyz=0.1 0 0 rpy=0 0 0 -> xyz=0.12 0 0 rpy=0 0 0
- joint left_delta_arm_joint: limit lower=-1.0471975511965976 upper=1.0471975511965976 effort=6 velocity=8 -> lower=-0.3490658503988659 upper=1.5707963267948966 effort=6 velocity=8; origin xyz=-0.05 0.0866 0 rpy=0 0 2.0943951023931953 -> xyz=-0.06 0.1039 0 rpy=0 0 2.0943951023931953
- joint right_delta_arm_joint: limit lower=-1.0471975511965976 upper=1.0471975511965976 effort=6 velocity=8 -> lower=-0.3490658503988659 upper=1.5707963267948966 effort=6 velocity=8; origin xyz=-0.05 -0.0866 0 rpy=0 0 -2.0943951023931953 -> xyz=-0.06 -0.1039 0 rpy=0 0 -2.0943951023931953

File: urdf/delta.urdf.xacro (robot description, xacro)
@@ -3,7 +3,12 @@
 <robot name="delta" xmlns:xacro="http://www.ros.org/wiki/xacro">
   <!-- Constants for robot dimensions -->
+  <xacro:property name="inch" value="0.0254"/>
   <xacro:property name="PI" value="3.1415926535897931"/>
   <xacro:property name="width" value="0.05" /> <!-- Square dimensions (widthxwidth) of beams -->
-  <xacro:property name="height1" value="0.05" /> <!-- base and end links -->
+  <xacro:property name="base_radius" value="0.111" />
+  <xacro:property name="base_length" value="${inch/2}"/>
+  <xacro:property name="platform_radius" value="0.0345" />
+  <xacro:property name="platform_length" value="${inch/4}"/>
+  <xacro:property name="platform_lower_link_dist" value="${platform_radius+0.03}"/>
   <xacro:include filename="macros.xacro" />
   <xacro:include filename="gazebo_stuff.xacro" />
@@ -17,26 +22,20 @@
   <link name="base_link">
     <collision>
-      <origin xyz="0 0 0" rpy="0 0 0"/>
+      <origin xyz="0 0 0" rpy="0 0 ${30*PI/180}"/>
       <geometry>
-	      <cylinder length="${height1}" radius="${height1*2}"/>
+        <cylinder radius="${base_radius}" length="${base_length}"/>
       </geometry>
     </collision>
     <visual>
-      <origin xyz="0 0 0" rpy="0 0 0"/>
+      <origin xyz="0 0 0" rpy="0 0 ${30*PI/180}"/>
       <geometry>
-	      <cylinder length="${height1}" radius="${height1*2}"/>
+        <mesh filename="file://$(find my_second_delta)/meshes/Base_Fija.stl" scale="0.001 0.001 0.001"/>
       </geometry>
-      <material name="orange">
-        <color rgba="${255/255} ${108/255} ${10/255} 1.0"/>
+      <material name="red">
       </material>
     </visual>
-    <inertial>
+    <xacro:inertial_cylinder mass="1.616" length="${base_length}" radius="${base_radius}">
       <origin xyz="0 0 0" rpy="0 0 0"/>
-      <mass value="1"/>
-      <inertia
-	      ixx="0.1" ixy="0.0" ixz="0.0"
-	      iyy="0.1" iyz="0.0"
-	      izz="0.1"/>
-    </inertial>
+    </xacro:inertial_cylinder>
   </link>
   <xacro:delta_arm prefix="front_"/>
@@ -44,8 +43,8 @@
     <parent link="base_link"/>
     <child link="front_upper_link"/>
-    <origin xyz="0.1 0 0" rpy="0 0 0"/>
+    <origin xyz="0.12 0 -0.0285" rpy="0 0 0"/>
     <axis xyz="0 1 0"/>
     <dynamics damping="0.7"/>
-    <limit lower="${-60*PI/180}" upper="${60*PI/180}" effort="6" velocity="8"/>
+    <limit lower="${-20*PI/180}" upper="${90*PI/180}" effort="6" velocity="8"/>
   </joint>
   <xacro:delta_arm prefix="right_"/>
@@ -53,8 +52,8 @@
     <parent link="base_link"/>
     <child link="right_upper_link"/>
-    <origin xyz="-0.05 -0.0866 0" rpy="0 0 ${-120*PI/180}"/>
+    <origin xyz="-0.06 -0.1039 -0.0285" rpy="0 0 ${-120*PI/180}"/>
     <axis xyz="0 1 0"/>
     <dynamics damping="0.7"/>
-    <limit lower="${-60*PI/180}" upper="${60*PI/180}" effort="6" velocity="8"/>
+    <limit lower="${-20*PI/180}" upper="${90*PI/180}" effort="6" velocity="8"/>
   </joint>
   <xacro:delta_arm prefix="left_"/>
@@ -62,38 +61,32 @@
     <parent link="base_link"/>
     <child link="left_upper_link"/>
-    <origin xyz="-0.05 0.0866 0" rpy="0 0 ${120*PI/180}"/>
+    <origin xyz="-0.06 0.1039 -0.0285" rpy="0 0 ${120*PI/180}"/>
     <axis xyz="0 1 0"/>
     <dynamics damping="0.7"/>
-    <limit lower="${-60*PI/180}" upper="${60*PI/180}" effort="6" velocity="8"/>
+    <limit lower="${-20*PI/180}" upper="${90*PI/180}" effort="6" velocity="8"/>
   </joint>
   <link name="end_link">
     <collision>
-      <origin xyz="0 0 0" rpy="0 0 0"/>
+      <origin xyz="0 0 0" rpy="0 0 ${-30*PI/180}"/>
       <geometry>
-	      <cylinder length="${height1/4}" radius="${height1/2}"/>
+	      <cylinder length="${platform_length}" radius="${platform_radius}"/>
       </geometry>
     </collision>
     <visual>
-      <origin xyz="0 0 0" rpy="0 0 0"/>
+      <origin xyz="0 0 0" rpy="0 0 ${-30*PI/180}"/>
       <geometry>
-	      <cylinder length="${height1/4}" radius="${height1/2}"/>
+        <mesh filename="file://$(find my_second_delta)/meshes/Base_Movil.stl" scale="0.001 0.001 0.001"/>
       </geometry>
-      <material name="orange">
-        <color rgba="${255/255} ${108/255} ${10/255} 1.0"/>
+      <material name="black">
       </material>
     </visual>
-    <inertial>
-      <origin xyz="0 0 0" rpy="0 0 0"/>
-      <mass value="0.1"/>
-      <inertia
-	      ixx="0.001" ixy="0.0" ixz="0.0"
-	      iyy="0.001" iyz="0.0"
-	      izz="0.001"/>
-    </inertial>
+    <xacro:inertial_cylinder mass="${mass}" length="${platform_length}" radius="${platform_radius}">
+      <origin xyz="0 0 0" rpy="0 0 ${-30*PI/180}"/>
+    </xacro:inertial_cylinder>
   </link>
   <joint name="front_end_joint" type="fixed">
     <parent link="front_lower_end_link"/>
     <child link="end_link"/>
-    <origin xyz="-0.05 0 0" rpy="0 0 0"/>
+    <origin xyz="-0.0645 0 0" rpy="0 0 0"/>
   </joint>
   <link name="right_end_virtual_link">
@@ -110,5 +103,5 @@
     <parent link="end_link"/>
     <child link="right_end_virtual_link"/>
-    <origin xyz="-0.025 -0.0433 0" rpy="0 0 ${-120*PI/180}"/>
+    <origin xyz="-0.017 -0.02785 0" rpy="0 0 ${-120*PI/180}"/>
   </joint>
   <link name="left_end_virtual_link">
@@ -125,5 +118,5 @@
     <parent link="end_link"/>
     <child link="left_end_virtual_link"/>
-    <origin xyz="-0.025 0.0433 0" rpy="0 0 ${120*PI/180}"/>
+    <origin xyz="-0.017 0.02785 0" rpy="0 0 ${120*PI/180}"/>
   </joint>
   <gazebo>

File: urdf/gazebo_stuff.xacro (robot description, xacro)
@@ -19,5 +19,5 @@
   </gazebo>
   <gazebo reference="end_link">
-    <material>Gazebo/Orange</material>
+    <material>Gazebo/Black</material>
     <selfCollide>false</selfCollide>
   </gazebo>
@@ -54,5 +54,5 @@
   <xacro:macro name="delta_arm_gazebo" params="prefix">
     <gazebo reference="${prefix}upper_link">
-      <material>Gazebo/Black</material>
+      <material>Gazebo/Grey</material>
       <selfCollide>false</selfCollide>
     </gazebo>
@@ -74,5 +74,5 @@
     </gazebo>
     <gazebo reference="${prefix}lower_end_link">
-      <material>Gazebo/Black</material>
+      <material>Gazebo/Red</material>
       <selfCollide>false</selfCollide>
     </gazebo>
@@ -140,4 +140,15 @@
   <material name="black">
     <color rgba="0.0 0.0 0.0 1.0"/>
+    <script>
+      <uri>file://media/materials/scripts/gazebo.material</uri>
+      <name>Gazebo/Black</name>
+    </script>
+    <shader type='pixel'>
+      <normal_map>__default__</normal_map>
+    </shader>
+    <ambient>0.3 0.3 0.3 1</ambient>
+    <diffuse>0.7 0.7 0.7 1</diffuse>
+    <specular>0.01 0.01 0.01 1</specular>
+    <emissive>0 0 0 1</emissive>
   </material>
   <material name="blue">
@@ -149,4 +160,15 @@
   <material name="grey">
     <color rgba="0.2 0.2 0.2 1.0"/>
+    <script>
+      <uri>file://media/materials/scripts/gazebo.material</uri>
+      <name>Gazebo/Red</name>
+    </script>
+    <shader type='pixel'>
+      <normal_map>__default__</normal_map>
+    </shader>
+    <ambient>0.3 0.3 0.3 1</ambient>
+    <diffuse>0.7 0.7 0.7 1</diffuse>
+    <specular>0.01 0.01 0.01 1</specular>
+    <emissive>0 0 0 1</emissive>
   </material>
   <material name="orange">
@@ -158,4 +180,15 @@
   <material name="red">
     <color rgba="0.8 0.0 0.0 1.0"/>
+    <script>
+      <uri>file://media/materials/scripts/gazebo.material</uri>
+      <name>Gazebo/Red</name>
+    </script>
+    <shader type='pixel'>
+      <normal_map>__default__</normal_map>
+    </shader>
+    <ambient>0.3 0.3 0.3 1</ambient>
+    <diffuse>0.7 0.7 0.7 1</diffuse>
+    <specular>0.01 0.01 0.01 1</specular>
+    <emissive>0 0 0 1</emissive>
   </material>
   <material name="white">

File: urdf/macros.xacro (robot description, xacro)
@@ -1,50 +1,73 @@
 <?xml version="1.0"?>
 <robot xmlns:xacro="http://www.ros.org/wiki/xacro">
+  <xacro:macro name="inertial_sphere" params="mass radius *origin">
+      <inertial>
+          <xacro:insert_block name="origin"/>
+          <mass value="${mass}"/>
+          <inertia ixx="${(2/5) * mass * (radius * radius)}" ixy="0.0" ixz="0.0"
+                  iyy="${(2/5) * mass * (radius * radius)}" iyz="0.0"
+                  izz="${(2/5) * mass * (radius * radius)}"/>
+      </inertial>
+  </xacro:macro>
+  <xacro:macro name="inertial_box" params="mass x y z *origin">
+      <inertial>
+          <xacro:insert_block name="origin"/>
+          <mass value="${mass}"/>
+          <inertia ixx="${(1/12) * mass * (y*y + z*z)}" ixy="0.0" ixz="0.0"
+                  iyy="${(1/12) * mass * (x*x + z*z)}" iyz="0.0"
+                  izz="${(1/12) * mass * (y*y + x*x)}"/>
+      </inertial>
+  </xacro:macro>
+  <xacro:macro name="inertial_cylinder" params="mass length radius *origin">
+      <inertial>
+          <xacro:insert_block name="origin"/>
+          <mass value="${mass}"/>
+          <inertia ixx="${(1/12) * mass * (3*radius*radius + length*length)}" ixy="0.0" ixz="0.0"
+                  iyy="${(1/12) * mass * (3*radius*radius + length*length)}" iyz="0.0"
+                  izz="${(1/2) * mass * (radius*radius)}"/>
+      </inertial>
+  </xacro:macro>
     <!-- Constants for robot dimensions -->
   <xacro:property name="PI" value="3.1415926535897931"/>
+  <xacro:property name="inch" value="0.0254"/>
   <!-- ==================================================================== -->
   <!-- ==================================================================== -->
   <!-- Important angle when robot at origin point, must be calculated!!!!!! -->
-  <xacro:property name="elbow_angle" value="${30*PI/180}" />
+  <xacro:property name="elbow_angle" value="${32.5*PI/180}" />
   <!-- ==================================================================== -->
   <!-- ==================================================================== -->
   <xacro:property name="wrist_angle" value="-${elbow_angle}" />
   <xacro:property name="mass" value="0.02" /> <!-- arbitrary value for mass -->
-  <xacro:property name="upper_width" value="0.04" /> <!-- Square dimensions (widthxwidth) of beams -->
+  <xacro:property name="upper_width" value="${inch/4}" /> <!-- Square dimensions (widthxwidth) of beams -->
+  <xacro:property name="upper_height" value="0.043"/>
   <xacro:property name="lower_width" value="0.01" />
-  <xacro:property name="upper_height" value="0.2" /> <!-- base and end links -->
+  <xacro:property name="upper_length" value="0.1475" /> <!-- base and end links -->
   <xacro:property name="lower_height1" value="0.06" /> <!-- Upper link -->
-  <xacro:property name="lower_height2" value="0.5" /> <!-- lower link -->
+  <xacro:property name="lower_height2" value="0.375" /> <!-- lower link -->
   <xacro:property name="lower_height3" value="0.03" /> <!-- Upper link -->
   <xacro:macro name="delta_arm" params="prefix">
     <link name="${prefix}upper_link">
       <collision>
-        <origin xyz="${upper_height/2} 0 0" rpy="0 0 0"/>
-        <geometry>
-          <box size="${upper_height} ${upper_width} ${upper_width}"/>
-        </geometry>
-      </collision>
-      <visual>
-        <origin xyz="${upper_height/2} 0 0" rpy="0 0 0"/>
-        <geometry>
-          <box size="${upper_height} ${upper_width} ${upper_width}"/>
-        </geometry>
-        <material name="black">
-          <color rgba="0.0 0.0 0.0 1.0"/>
-        </material>
-      </visual>
-      <inertial>
-        <origin xyz="0 0 ${upper_height/2}" rpy="0 0 0"/>
-        <mass value="${mass}"/>
-        <inertia
-          ixx="${mass / 12.0 * (upper_width*upper_width + upper_width*upper_width)}" ixy="0.0" ixz="0.0"
-          iyy="${mass / 12.0 * (upper_height*upper_height + upper_width*upper_width)}" iyz="0.0"
-          izz="${mass / 12.0 * (upper_height*upper_height + upper_width*upper_width)}"/>
-      </inertial>
+        <origin xyz="0 0 0" rpy="0 0 0"/>
+        <geometry>
+          <box size="${upper_length} ${upper_width} ${upper_height}"/>
+        </geometry>
+      </collision>
+      <visual>
+        <origin xyz="0 0 0" rpy="0 0 0"/>
+        <geometry>
+          <mesh filename="file://$(find my_second_delta)/meshes/Brazo.stl" scale="0.001 0.001 0.001"/>
+        </geometry>
+        <material name="grey">
+        </material>
+      </visual>
+      <xacro:inertial_box mass="${mass}" x="${upper_length}" y="${upper_width}" z="${upper_height}">
+        <origin xyz="0 0 0" rpy="0 0 0"/>
+      </xacro:inertial_box>
     </link>
     <joint name="${prefix}upper_joint" type="continuous">
       <parent link="${prefix}upper_link"/>
       <child link="${prefix}lower_top_link"/>
-      <origin xyz="${upper_height} 0 0" rpy="0 ${elbow_angle} 0"/>
+      <origin xyz="${upper_length} 0 0" rpy="0 ${elbow_angle} 0"/>
       <axis xyz="0 1 0"/>
     </joint>
