Commit message: RDS_w/nodes

File: urdf/macros.xacro (robot description, xacro)
@@ -49,5 +49,5 @@
     <link name="${prefix}upper_link">
       <collision>
-        <origin xyz="0 0 0" rpy="0 0 0"/>
+        <origin xyz="0 0 0" rpy="${180*PI/180} 0 0"/>
         <geometry>
           <box size="${upper_length} ${upper_width} ${upper_height}"/>
@@ -55,5 +55,5 @@
       </collision>
       <visual>
-        <origin xyz="0 0 0" rpy="0 0 0"/>
+        <origin xyz="0 0 0" rpy="${180*PI/180} 0 0"/>
         <geometry>
           <mesh filename="file://$(find my_second_delta)/meshes/Brazo.stl" scale="0.001 0.001 0.001"/>
@@ -63,5 +63,5 @@
       </visual>
       <xacro:inertial_box mass="${mass}" x="${upper_length}" y="${upper_width}" z="${upper_height}">
-        <origin xyz="0 0 0" rpy="0 0 0"/>
+        <origin xyz="0 0 0" rpy="${180*PI/180} 0 0"/>
       </xacro:inertial_box>
     </link>
