Commit message: Second Commit

File: urdf/delta.urdf.xacro (robot description, xacro)
@@ -1,28 +1,13 @@
 <?xml version="1.0"?>
 <robot xmlns:xacro="http://www.ros.org/wiki/xacro" name="delta">
+    <xacro:property name="PI" value="3.1415926535897931"/>
+    <xacro:property name="inch" value="0.0254"/>
+    <xacro:property name="base_radius" value="0.111" /> <!-- Square dimensions (widthxwidth) of beams -->
+    <xacro:property name="base_height" value="${inch/2}" /> <!-- base and end links -->
     <xacro:include filename="macros.xacro"/>
-    <xacro:property name="inch" value="0.0254"/>
+    <!-- Include gazebo plugins -->
+    <xacro:include filename="gazebo_stuff.xacro" />
     <!-- Base of the robot -->
     <link name="world"/>
-    <link name="base_link">
-        <visual>
-            <origin xyz="0.0 0.0 ${inch/4}"/>
-            <geometry>
-                <cylinder radius="0.111" length="${inch/2}"/>
-            </geometry>
-            <material name="green">
-                <color rgba="0.2 1 0.2 1"/>
-            </material>
-        </visual>
-        <collision>
-            <origin xyz="0.0 0.0 ${inch/4}"/>
-            <geometry>
-                <cylinder radius="0.111" length="${inch/2}"/>
-            </geometry>
-        </collision>
-        <xacro:inertial_cylinder mass="12" length="${inch/2}" radius="0.111">
-            <origin xyz="0.0 0.0 ${inch/4}"/>
-        </xacro:inertial_cylinder>
-    </link>
     <joint name="world_base_joint" type="fixed">
         <origin xyz="1 0.0 0.0" rpy="0.0 0.0 0.0"/>
@@ -30,236 +15,51 @@
         <child link="base_link"/>
     </joint>
-    <!-- First Arm -->
-    <link name="arm_1_link">
+    <link name="base_link">
         <visual>
-            <origin xyz="-0.09 0.0 0.0" rpy="0.0 0.0 0.0"/>
+            <origin xyz="0.0 0.0 0.0" rpy="0.0 0.0 0.0"/>
             <geometry>
-                <box size="0.185 ${inch/4} 0.043"/>
+                <cylinder radius="${base_radius}" length="${base_height}"/>
             </geometry>
-            <material name="green"/>
+            <material name="orange">
+                <color rgba="${255/255} ${108/255} ${10/255} 1.0"/>
+            </material>
         </visual>
         <collision>
-            <origin xyz="-0.09 0.0 0.0" rpy="0.0 0.0 0.0"/>
+            <origin xyz="0.0 0.0 0.0" rpy="0.0 0.0 0.0"/>
             <geometry>
-                <box size="0.185 ${inch/4} 0.043"/>
+                <cylinder radius="${base_radius}" length="${base_height}"/>
             </geometry>
         </collision>
-        <xacro:inertial_box mass="6" x="0.185" y="${inch/4}" z="0.043">
-            <origin xyz="-0.09 0.0 0.0" rpy="0.0 0.0 0.0"/>
-        </xacro:inertial_box>
+        <xacro:inertial_cylinder mass="12" length="${base_height}" radius="${base_radius}">
+            <origin xyz="0.0 0.0 0.0" rpy="0.0 0.0 0.0"/>
+        </xacro:inertial_cylinder>
     </link>
-    <joint name="base_arm_1_joint" type="revolute">
-        <origin xyz="-0.115 0.0 ${inch}" rpy="0.0 0.0 0.0"/>
+    <xacro:delta_arm prefix="1"/>
+    <joint name="arm_1_delta_joint" type="revolute">
         <parent link="base_link"/>
         <child link="arm_1_link"/>
-        <axis xyz="0.0 1.0 0.0"/>
-        <limit lower="${-pi/2}" upper="${pi/2}" effort="100.0" velocity="100.0"/>
-        <dynamics damping="4" friction="4" />
+        <origin xyz="${base_radius} 0.0 0.0" rpy="0.0 0.0 0.0"/>
+        <axis xyz="0.0 1 0.0"/>
+        <dynamics damping="0.7"/>
+        <limit lower="${-20*PI/180}" upper="${90*PI/180}" effort="6" velocity="8"/>
     </joint>
-    <!-- Second Arm -->
-    <link name="arm_2_link">
-        <visual>
-            <origin xyz="-0.09 0.0 0.0" rpy="0.0 0.0 0.0"/>
-            <geometry>
-                <box size="0.185 ${inch/4} 0.043"/>
-            </geometry>
-            <material name="green"/>
-        </visual>
-        <collision>
-            <origin xyz="-0.09 0.0 0.0" rpy="0.0 0.0 0.0"/>
-            <geometry>
-                <box size="0.185 ${inch/4} 0.043"/>
-            </geometry>
-        </collision>
-        <xacro:inertial_box mass="6" x="0.185" y="${inch/4}" z="0.043">
-            <origin xyz="-0.09 0.0 0.0" rpy="0.0 0.0 0.0"/>
-        </xacro:inertial_box>
-    </link>
-    <joint name="base_arm_2_joint" type="revolute">
-        <origin xyz="0.055 0.096 ${inch}" rpy="0.0 0.0 ${-120*pi/180}"/>
+    <xacro:delta_arm prefix="2"/>
+    <joint name="arm_2_delta_joint" type="revolute">
         <parent link="base_link"/>
         <child link="arm_2_link"/>
-        <axis xyz="0.0 1.0 0.0"/>
-        <limit lower="${-pi/2}" upper="${pi/2}" effort="100.0" velocity="100.0"/>
-        <dynamics damping="4" friction="4" />
+        <origin xyz="-0.0555 0.09612 0.0" rpy="0.0 0.0 ${-120*PI/180}"/>
+        <axis xyz="0.0 1 0.0"/>
+        <dynamics damping="0.7"/>
+        <limit lower="${-20*PI/180}" upper="${90*PI/180}" effort="6" velocity="8"/>
     </joint>
-    <!-- Third Arm -->
-    <link name="arm_3_link">
-        <visual>
-            <origin xyz="-0.09 0.0 0.0" rpy="0.0 0.0 0.0"/>
-            <geometry>
-                <box size="0.185 ${inch/4} 0.043"/>
-            </geometry>
-            <material name="green"/>
-        </visual>
-        <collision>
-            <origin xyz="-0.09 0.0 0.0" rpy="0.0 0.0 0.0"/>
-            <geometry>
-                <box size="0.185 ${inch/4} 0.043"/>
-            </geometry>
-        </collision>
-        <xacro:inertial_box mass="6" x="0.185" y="${inch/4}" z="0.043">
-            <origin xyz="-0.09 0.0 0.0" rpy="0.0 0.0 0.0"/>
-        </xacro:inertial_box>
-    </link>
-    <joint name="base_arm_3_joint" type="revolute">
-        <origin xyz="0.055 -0.096 ${inch}" rpy="0.0 0.0 ${120*pi/180}"/>
+    <xacro:delta_arm prefix="3"/>
+    <joint name="arm_3_delta_joint" type="revolute">
         <parent link="base_link"/>
         <child link="arm_3_link"/>
-        <axis xyz="0.0 1.0 0.0"/>
-        <limit lower="${-pi/2}" upper="${pi/2}" effort="100.0" velocity="100.0"/>
-        <dynamics damping="4" friction="4" />
+        <origin xyz="-0.0555 -0.09612 0.0" rpy="0.0 0.0 ${120*PI/180}"/>
+        <axis xyz="0.0 1 0.0"/>
+        <dynamics damping="0.7"/>
+        <limit lower="${-20*PI/180}" upper="${90*PI/180}" effort="6" velocity="8"/>
     </joint>
-    <!-- Forearm 1 -->
-    <link name="forearm_1_link">
-        <visual>
-            <origin xyz="0.0 0.0 0.175" rpy="0.0 0.0 0.0"/>
-            <geometry>
-                <cylinder radius="${inch/4}" length="0.350"/>
-            </geometry>
-            <material name="green"/>
-        </visual>
-        <collision>
-            <origin xyz="0.0 0.0 0.175" rpy="0.0 0.0 0.0"/>
-            <geometry>
-                <cylinder radius="${inch/4}" length="0.350"/>
-            </geometry>
-        </collision>
-        <xacro:inertial_cylinder mass="4" length="${inch/4}" radius="0.350">
-            <origin xyz="0.0 0.0 0.0"/>
-        </xacro:inertial_cylinder>
-    </link>
-    <!-- Spherical Joint 1 -->
-    <link name="virtual_link_1_1">
-        <xacro:inertial_box mass="0.1" x="0.01" y="0.01" z="0.01">
-            <origin xyz="0.0 0.0 0.0"/>
-        </xacro:inertial_box>
-    </link>
-    <link name="virtual_link_1_2">
-        <xacro:inertial_box mass="0.1" x="0.01" y="0.01" z="0.01">
-            <origin xyz="0.0 0.0 0.0"/>
-        </xacro:inertial_box>
-    </link>
-    <joint name="arm_forearm_1_1_joint" type="revolute">
-        <origin xyz="-0.190 0.0 0.0" rpy="0.0 0.0 0.0"/>
-        <parent link="arm_1_link"/>
-        <child link="virtual_link_1_1"/>
-        <axis xyz="1.0 0.0 0.0"/>
-        <limit lower="${-24*pi/180}" upper="${24*pi/180}" effort="100.0" velocity="100.0"/>
-        <dynamics friction="0.003" damping="0.0"/>
-    </joint>
-    <joint name="arm_forearm_1_2_joint" type="revolute">
-        <parent link="virtual_link_1_1"/>
-        <child link="virtual_link_1_2"/>
-        <axis xyz="0.0 1.0 0.0"/>
-        <limit lower="${-pi}" upper="${pi}" effort="100.0" velocity="100.0"/>
-        <dynamics friction="0.003" damping="0.0"/>
-    </joint>
-    <joint name="arm_forearm_1_3_joint" type="revolute">
-        <parent link="virtual_link_1_2"/>
-        <child link="forearm_1_link"/>
-        <axis xyz="0.0 0.0 1.0"/>
-        <limit lower="${-24*pi/180}" upper="${24*pi/180}" effort="100.0" velocity="100.0"/>
-        <dynamics friction="0.003" damping="0.0"/>
-    </joint>
-    <!-- Forearm 2 -->
-    <link name="forearm_2_link">
-        <visual>
-            <origin xyz="0.0 0.0 0.175" rpy="0.0 0.0 0.0"/>
-            <geometry>
-                <cylinder radius="${inch/4}" length="0.350"/>
-            </geometry>
-            <material name="green"/>
-        </visual>
-        <collision>
-            <origin xyz="0.0 0.0 0.175" rpy="0.0 0.0 0.0"/>
-            <geometry>
-                <cylinder radius="${inch/4}" length="0.350"/>
-            </geometry>
-        </collision>
-        <xacro:inertial_cylinder mass="4" length="${inch/4}" radius="0.350">
-            <origin xyz="0.0 0.0 0.0"/>
-        </xacro:inertial_cylinder>
-    </link>
-    <!-- Spherical Joint 2 -->
-    <link name="virtual_link_2_1">
-        <xacro:inertial_box mass="0.1" x="0.01" y="0.01" z="0.01">
-            <origin xyz="0.0 0.0 0.0"/>
-        </xacro:inertial_box>
-    </link>
-    <link name="virtual_link_2_2">
-        <xacro:inertial_box mass="0.1" x="0.01" y="0.01" z="0.01">
-            <origin xyz="0.0 0.0 0.0"/>
-        </xacro:inertial_box>
-    </link>
-    <joint name="arm_forearm_2_1_joint" type="revolute">
-        <origin xyz="-0.190 0.0 0.0" rpy="0.0 0.0 0.0"/>
-        <parent link="arm_2_link"/>
-        <child link="virtual_link_2_1"/>
-        <axis xyz="1.0 0.0 0.0"/>
-        <limit lower="${-24*pi/180}" upper="${24*pi/180}" effort="100.0" velocity="100.0"/>
-    </joint>
-    <joint name="arm_forearm_2_2_joint" type="revolute">
-        <parent link="virtual_link_2_1"/>
-        <child link="virtual_link_2_2"/>
-        <axis xyz="0.0 1.0 0.0"/>
-        <limit lower="${-pi}" upper="${pi}" effort="100.0" velocity="100.0"/>
-    </joint>
-    <joint name="arm_forearm_2_3_joint" type="revolute">
-        <parent link="virtual_link_2_2"/>
-        <child link="forearm_2_link"/>
-        <axis xyz="0.0 0.0 1.0"/>
-        <limit lower="${-24*pi/180}" upper="${24*pi/180}" effort="100.0" velocity="100.0"/>
-    </joint>
-    <!-- Forearm 3 -->
-    <link name="forearm_3_link">
-        <visual>
-            <origin xyz="0.0 0.0 0.175" rpy="0.0 0.0 0.0"/>
-            <geometry>
-                <cylinder radius="${inch/4}" length="0.350"/>
-            </geometry>
-            <material name="green"/>
-        </visual>
-        <collision>
-            <origin xyz="0.0 0.0 0.175" rpy="0.0 0.0 0.0"/>
-            <geometry>
-                <cylinder radius="${inch/4}" length="0.350"/>
-            </geometry>
-        </collision>
-        <xacro:inertial_cylinder mass="4" length="${inch/4}" radius="0.350">
-            <origin xyz="0.0 0.0 0.0"/>
-        </xacro:inertial_cylinder>
-    </link>
-    <!-- Spherical Joint 3 -->
-    <link name="virtual_link_3_1">
-        <xacro:inertial_box mass="0.1" x="0.01" y="0.01" z="0.01">
-            <origin xyz="0.0 0.0 0.0"/>
-        </xacro:inertial_box>
-    </link>
-    <link name="virtual_link_3_2">
-        <xacro:inertial_box mass="0.1" x="0.01" y="0.01" z="0.01">
-            <origin xyz="0.0 0.0 0.0"/>
-        </xacro:inertial_box>
-    </link>
-    <joint name="arm_forearm_3_1_joint" type="revolute">
-        <origin xyz="-0.190 0.0 0.0" rpy="0.0 0.0 0.0"/>
-        <parent link="arm_3_link"/>
-        <child link="virtual_link_3_1"/>
-        <axis xyz="1.0 0.0 0.0"/>
-        <limit lower="${-24*pi/180}" upper="${24*pi/180}" effort="100.0" velocity="100.0"/>
-    </joint>
-    <joint name="arm_forearm_3_2_joint" type="revolute">
-        <parent link="virtual_link_3_1"/>
-        <child link="virtual_link_3_2"/>
-        <axis xyz="0.0 1.0 0.0"/>
-        <limit lower="${-pi}" upper="${pi}" effort="100.0" velocity="100.0"/>
-    </joint>
-    <joint name="arm_forearm_3_3_joint" type="revolute">
-        <parent link="virtual_link_3_2"/>
-        <child link="forearm_3_link"/>
-        <axis xyz="0.0 0.0 1.0"/>
-        <limit lower="${-24*pi/180}" upper="${24*pi/180}" effort="100.0" velocity="100.0"/>
-    </joint>
-    <!-- Mobile Platform -->
     <link name="mobile_platform">
         <visual>
@@ -267,6 +67,7 @@
                 <cylinder radius="0.035" length="${inch/4}"/>
             </geometry>
-            <origin xyz="0.0 0.0 -${inch/8}"/>
-            <material name="green">
+            <origin xyz="0.0 0.0 0.0" rpy="0.0 0.0 0.0"/>
+            <material name="orange">
+                <color rgba="${255/255} ${108/255} ${10/255} 1.0"/>
             </material>
         </visual>
@@ -275,75 +76,56 @@
                 <cylinder radius="0.035" length="${inch/4}"/>
             </geometry>
-            <origin xyz="0.0 0.0 -${inch/8}"/>
+            <origin xyz="0.0 0.0 0.0" rpy="0.0 0.0 0.0"/>
         </collision>
-        <xacro:inertial_cylinder mass="4" length="${inch/4}" radius="0.035">
-            <origin xyz="0.0 0.0 -${inch/8}"/>
+        <xacro:inertial_cylinder mass="0.1" length="${inch/4}" radius="0.035">
+            <origin xyz="0.0 0.0 0.0" rpy="0.0 0.0 0.0"/>
         </xacro:inertial_cylinder>
     </link>
-    <!-- Spherical Joint 4 -->
-    <link name="virtual_link_1_4">
-        <xacro:inertial_box mass="0.1" x="0.01" y="0.01" z="0.01">
-            <origin xyz="0.0 0.0 0.0"/>
-        </xacro:inertial_box>
+    <joint name="1_mobile_joint" type="fixed">
+        <parent link="forearm_1_end_link"/>
+        <child link="mobile_platform"/>
+        <origin xyz="-0.035 0 0" rpy="0 0 0"/>
+    </joint>
+    <link name="2_mobile_virtual_link">
+        <inertial>
+        <origin xyz="0 0 0" rpy="0 0 0"/>
+        <mass value="0.001"/>
+        <inertia
+            ixx="0.0001" ixy="0.0" ixz="0.0"
+            iyy="0.0001" iyz="0.0"
+            izz="0.0001"/>
+        </inertial>
     </link>
-    <link name="virtual_link_1_5">
-        <xacro:inertial_box mass="0.1" x="0.01" y="0.01" z="0.01">
-            <origin xyz="0.0 0.0 0.0"/>
-        </xacro:inertial_box>
+    <joint name="2_mobile_virtual_joint" type="fixed">
+        <parent link="mobile_platform"/>
+        <child link="2_mobile_virtual_link"/>
+        <origin xyz="0.0175 -0.03031 0" rpy="0 0 ${-120*PI/180}"/>
+    </joint>
+    <link name="3_mobile_virtual_link">
+        <inertial>
+        <origin xyz="0 0 0" rpy="0 0 0"/>
+        <mass value="0.001"/>
+        <inertia
+            ixx="0.0001" ixy="0.0" ixz="0.0"
+            iyy="0.0001" iyz="0.0"
+            izz="0.0001"/>
+        </inertial>
     </link>
-    <joint name="arm_forearm_1_4_joint" type="revolute">
-        <origin xyz="0.0 0.0 ${0.350+inch/4}" rpy="0.0 0.0 0.0"/>
-        <parent link="forearm_1_link"/>
-        <child link="virtual_link_1_4"/>
-        <axis xyz="1.0 0.0 0.0"/>
-        <limit lower="${-24*pi/180}" upper="${24*pi/180}" effort="100.0" velocity="100.0"/>
-    </joint>
-    <joint name="arm_forearm_1_5_joint" type="revolute">
-        <parent link="virtual_link_1_4"/>
-        <child link="virtual_link_1_5"/>
-        <axis xyz="0.0 1.0 0.0"/>
-        <limit lower="${-pi}" upper="${pi}" effort="100.0" velocity="100.0"/>
-    </joint>
-    <joint name="arm_forearm_1_6_joint" type="revolute">
-        <origin xyz="-0.035 0.0 0.0"/>
-        <parent link="virtual_link_1_5"/>
-        <child link="mobile_platform"/>
-        <axis xyz="0.0 0.0 1.0"/>
-        <limit lower="${-24*pi/180}" upper="${24*pi/180}" effort="100.0" velocity="100.0"/>
-    </joint>
-    <!-- Spherical Joint 5 -->
-    <link name="virtual_link_2_4">
-        <xacro:inertial_box mass="0.1" x="0.01" y="0.01" z="0.01">
-            <origin xyz="0.0 0.0 0.0"/>
-        </xacro:inertial_box>
-    </link>
-    <link name="virtual_link_2_5">
-        <xacro:inertial_box mass="0.1" x="0.01" y="0.01" z="0.01">
-            <origin xyz="0.0 0.0 0.0"/>
-        </xacro:inertial_box>
-    </link>
-    <joint name="arm_forearm_2_4_joint" type="revolute">
-        <origin xyz="0.0 0.0 ${0.350+inch/4}" rpy="0.0 0.0 0.0"/>
-        <parent link="forearm_2_link"/>
-        <child link="virtual_link_2_4"/>
-        <axis xyz="1.0 0.0 0.0"/>
-        <limit lower="${-24*pi/180}" upper="${24*pi/180}" effort="100.0" velocity="100.0"/>
-    </joint>
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
File: urdf/gazebo_stuff.xacro (robot description, xacro)
@@ -1,34 +1,54 @@
 <?xml version="1.0"?>
 <robot xmlns:xacro="http://www.ros.org/wiki/xacro">
-    <gazebo reference="base_link">
-        <material>Gazebo/Green</material>
-    </gazebo>
+    <physics type='ode'>
+        <max_step_size>0.001</max_step_size>
+        <real_time_factor>0.1</real_time_factor>
+        <real_time_update_rate>1000</real_time_update_rate>
+        <gravity>0 0 -9.8</gravity>
+    </physics>
     <gazebo>
-        <plugin name="gazebo_ros_joint_state_publisher" filename="libgazebo_ros_joint_state_publisher.so">
-            <update_rate>20</update_rate>
-            <joint_name>base_arm_1_joint</joint_name>
-            <joint_name>arm_forearm_1_1_joint</joint_name>
-            <joint_name>arm_forearm_1_2_joint</joint_name>
-            <joint_name>arm_forearm_1_3_joint</joint_name>
-            <joint_name>arm_forearm_1_4_joint</joint_name>
-            <joint_name>arm_forearm_1_5_joint</joint_name>
-            <joint_name>arm_forearm_1_6_joint</joint_name>
-            <joint_name>base_arm_2_joint</joint_name>
-            <joint_name>arm_forearm_2_1_joint</joint_name>
-            <joint_name>arm_forearm_2_2_joint</joint_name>
-            <joint_name>arm_forearm_2_3_joint</joint_name>
-            <joint_name>arm_forearm_2_4_joint</joint_name>
-            <joint_name>arm_forearm_2_5_joint</joint_name>
-            <joint_name>arm_forearm_2_6_joint</joint_name>
-            <joint_name>base_arm_3_joint</joint_name>
-            <joint_name>arm_forearm_3_1_joint</joint_name>
-            <joint_name>arm_forearm_3_2_joint</joint_name>
-            <joint_name>arm_forearm_3_3_joint</joint_name>
+        <plugin name="gazebo_ros_control" filename="libgazebo_ros_control.so">
+        <robotNamespace></robotNamespace>
+        <robotSimType>gazebo_ros_control/DefaultRobotHWSim</robotSimType>
+        <legacyModeNS>true</legacyModeNS>
         </plugin>
     </gazebo>
-    <gazebo>
-        <plugin name="gazebo_ros_joint_pose_trajectory" filename="libgazebo_ros_joint_pose_trajectory.so">
-            <update_rate>20</update_rate>
-        </plugin>
+    <gazebo reference="base_link">
+        <material>Gazebo/Orange</material>
+        <selfCollide>false</selfCollide>
     </gazebo>
+    <gazebo reference="end_link">
+        <material>Gazebo/Orange</material>
+        <selfCollide>false</selfCollide>
+    </gazebo>
+    <transmission name="arm_1_delta_joint_trans">
+        <type>transmission_interface/SimpleTransmission</type>
+        <joint name="arm_1_delta_joint">
+        <hardwareInterface>hardware_interface/EffortJointInterface</hardwareInterface>
+        </joint>
+        <actuator name="arm_1_delta_joint_motor">
+        <hardwareInterface>hardware_interface/EffortJointInterface</hardwareInterface>
+        <mechanicalReduction>1</mechanicalReduction>
+        </actuator>
+    </transmission>
+    <transmission name="arm_2_delta_joint_trans">
+        <type>transmission_interface/SimpleTransmission</type>
+        <joint name="arm_2_delta_joint">
+        <hardwareInterface>hardware_interface/EffortJointInterface</hardwareInterface>
+        </joint>
+        <actuator name="arm_2_delta_joint_motor">
+        <hardwareInterface>hardware_interface/EffortJointInterface</hardwareInterface>
+        <mechanicalReduction>1</mechanicalReduction>
+        </actuator>
+    </transmission>
+    <transmission name="arm_3_delta_joint_trans">
+        <type>transmission_interface/SimpleTransmission</type>
+        <joint name="arm_3_delta_joint">
+        <hardwareInterface>hardware_interface/EffortJointInterface</hardwareInterface>
+        </joint>
+        <actuator name="arm_3_delta_joint_motor">
+        <hardwareInterface>hardware_interface/EffortJointInterface</hardwareInterface>
+        <mechanicalReduction>1</mechanicalReduction>
+        </actuator>
+    </transmission>
 </robot>
