Commit message: Delta Working in Gazebo

File: urdf/delta.urdf.xacro (robot description, xacro)
@@ -1,131 +1,141 @@
 <?xml version="1.0"?>
-<robot xmlns:xacro="http://www.ros.org/wiki/xacro" name="delta">
-    <xacro:property name="PI" value="3.1415926535897931"/>
-    <xacro:property name="inch" value="0.0254"/>
-    <xacro:property name="base_radius" value="0.111" /> <!-- Square dimensions (widthxwidth) of beams -->
-    <xacro:property name="base_height" value="${inch/2}" /> <!-- base and end links -->
-    <xacro:include filename="macros.xacro"/>
-    <!-- Include gazebo plugins -->
-    <xacro:include filename="gazebo_stuff.xacro" />
-    <!-- Base of the robot -->
-    <link name="world"/>
-    <joint name="world_base_joint" type="fixed">
-        <origin xyz="1 0.0 0.0" rpy="0.0 0.0 0.0"/>
-        <parent link="world"/>
-        <child link="base_link"/>
+<!-- Revolute-Revolute Manipulator -->
+<robot name="delta" xmlns:xacro="http://www.ros.org/wiki/xacro">
+  <!-- Constants for robot dimensions -->
+  <xacro:property name="PI" value="3.1415926535897931"/>
+  <xacro:property name="width" value="0.05" /> <!-- Square dimensions (widthxwidth) of beams -->
+  <xacro:property name="height1" value="0.05" /> <!-- base and end links -->
+  <xacro:include filename="macros.xacro" />
+  <xacro:include filename="gazebo_stuff.xacro" />
+  <!-- Used for fixing robot to Gazebo 'base_link' -->
+  <link name="world"/>
+  <joint name="fixed" type="fixed">
+    <parent link="world"/>
+    <child link="base_link"/>
+    <origin xyz="0 0 2" rpy="0 0 0"/>
+  </joint>
+  <link name="base_link">
+    <collision>
+      <origin xyz="0 0 0" rpy="0 0 0"/>
+      <geometry>
+	      <cylinder length="${height1}" radius="${height1*2}"/>
+      </geometry>
+    </collision>
+    <visual>
+      <origin xyz="0 0 0" rpy="0 0 0"/>
+      <geometry>
+	      <cylinder length="${height1}" radius="${height1*2}"/>
+      </geometry>
+      <material name="orange">
+        <color rgba="${255/255} ${108/255} ${10/255} 1.0"/>
+      </material>
+    </visual>
+    <inertial>
+      <origin xyz="0 0 0" rpy="0 0 0"/>
+      <mass value="1"/>
+      <inertia
+	      ixx="0.1" ixy="0.0" ixz="0.0"
+	      iyy="0.1" iyz="0.0"
+	      izz="0.1"/>
+    </inertial>
+  </link>
+  <xacro:delta_arm prefix="front_"/>
+  <joint name="front_delta_arm_joint" type="revolute">
+    <parent link="base_link"/>
+    <child link="front_upper_link"/>
+    <origin xyz="0.1 0 0" rpy="0 0 0"/>
+    <axis xyz="0 1 0"/>
+    <dynamics damping="0.7"/>
+    <limit lower="${-60*PI/180}" upper="${60*PI/180}" effort="6" velocity="8"/>
+  </joint>
+  <xacro:delta_arm prefix="right_"/>
+  <joint name="right_delta_arm_joint" type="revolute">
+    <parent link="base_link"/>
+    <child link="right_upper_link"/>
+    <origin xyz="-0.05 -0.0866 0" rpy="0 0 ${-120*PI/180}"/>
+    <axis xyz="0 1 0"/>
+    <dynamics damping="0.7"/>
+    <limit lower="${-60*PI/180}" upper="${60*PI/180}" effort="6" velocity="8"/>
+  </joint>
+  <xacro:delta_arm prefix="left_"/>
+  <joint name="left_delta_arm_joint" type="revolute">
+    <parent link="base_link"/>
+    <child link="left_upper_link"/>
+    <origin xyz="-0.05 0.0866 0" rpy="0 0 ${120*PI/180}"/>
+    <axis xyz="0 1 0"/>
+    <dynamics damping="0.7"/>
+    <limit lower="${-60*PI/180}" upper="${60*PI/180}" effort="6" velocity="8"/>
+  </joint>
+  <link name="end_link">
+    <collision>
+      <origin xyz="0 0 0" rpy="0 0 0"/>
+      <geometry>
+	      <cylinder length="${height1/4}" radius="${height1/2}"/>
+      </geometry>
+    </collision>
+    <visual>
+      <origin xyz="0 0 0" rpy="0 0 0"/>
+      <geometry>
+	      <cylinder length="${height1/4}" radius="${height1/2}"/>
+      </geometry>
+      <material name="orange">
+        <color rgba="${255/255} ${108/255} ${10/255} 1.0"/>
+      </material>
+    </visual>
+    <inertial>
+      <origin xyz="0 0 0" rpy="0 0 0"/>
+      <mass value="0.1"/>
+      <inertia
+	      ixx="0.001" ixy="0.0" ixz="0.0"
+	      iyy="0.001" iyz="0.0"
+	      izz="0.001"/>
+    </inertial>
+  </link>
+  <joint name="front_end_joint" type="fixed">
+    <parent link="front_lower_end_link"/>
+    <child link="end_link"/>
+    <origin xyz="-0.05 0 0" rpy="0 0 0"/>
+  </joint>
+  <link name="right_end_virtual_link">
+    <inertial>
+      <origin xyz="0 0 0" rpy="0 0 0"/>
+      <mass value="0.001"/>
+      <inertia
+        ixx="0.0001" ixy="0.0" ixz="0.0"
+        iyy="0.0001" iyz="0.0"
+        izz="0.0001"/>
+    </inertial>
+  </link>
+  <joint name="right_end_virtual_joint" type="fixed">
+    <parent link="end_link"/>
+    <child link="right_end_virtual_link"/>
+    <origin xyz="-0.025 -0.0433 0" rpy="0 0 ${-120*PI/180}"/>
+  </joint>
+  <link name="left_end_virtual_link">
+    <inertial>
+      <origin xyz="0 0 0" rpy="0 0 0"/>
+      <mass value="0.001"/>
+      <inertia
+        ixx="0.0001" ixy="0.0" ixz="0.0"
+        iyy="0.0001" iyz="0.0"
+        izz="0.0001"/>
+    </inertial>
+  </link>
+  <joint name="left_end_virtual_joint" type="fixed">
+    <parent link="end_link"/>
+    <child link="left_end_virtual_link"/>
+    <origin xyz="-0.025 0.0433 0" rpy="0 0 ${120*PI/180}"/>
+  </joint>
+  <gazebo>
+    <joint name="right_end_joint" type="fixed">
+      <parent>right_lower_end_link</parent>
+      <child>right_end_virtual_link</child>
+      <pose> 0 0 0 0 0 0 </pose>
     </joint>
-    <link name="base_link">
-        <visual>
-            <origin xyz="0.0 0.0 0.0" rpy="0.0 0.0 0.0"/>
-            <geometry>
-                <cylinder radius="${base_radius}" length="${base_height}"/>
-            </geometry>
-            <material name="orange">
-                <color rgba="${255/255} ${108/255} ${10/255} 1.0"/>
-            </material>
-        </visual>
-        <collision>
-            <origin xyz="0.0 0.0 0.0" rpy="0.0 0.0 0.0"/>
-            <geometry>
-                <cylinder radius="${base_radius}" length="${base_height}"/>
-            </geometry>
-        </collision>
-        <xacro:inertial_cylinder mass="12" length="${base_height}" radius="${base_radius}">
-            <origin xyz="0.0 0.0 0.0" rpy="0.0 0.0 0.0"/>
-        </xacro:inertial_cylinder>
-    </link>
-    <xacro:delta_arm prefix="1"/>
-    <joint name="arm_1_delta_joint" type="revolute">
-        <parent link="base_link"/>
-        <child link="arm_1_link"/>
-        <origin xyz="${base_radius} 0.0 0.0" rpy="0.0 0.0 0.0"/>
-        <axis xyz="0.0 1 0.0"/>
-        <dynamics damping="0.7"/>
-        <limit lower="${-20*PI/180}" upper="${90*PI/180}" effort="6" velocity="8"/>
+    <joint name="left_end_joint" type="fixed">
+      <parent>left_lower_end_link</parent>
+      <child>left_end_virtual_link</child>
+      <pose> 0 0 0 0 0 0 </pose>
     </joint>
-    <xacro:delta_arm prefix="2"/>
-    <joint name="arm_2_delta_joint" type="revolute">
-        <parent link="base_link"/>
-        <child link="arm_2_link"/>
-        <origin xyz="-0.0555 0.09612 0.0" rpy="0.0 0.0 ${-120*PI/180}"/>
-        <axis xyz="0.0 1 0.0"/>
-        <dynamics damping="0.7"/>
-        <limit lower="${-20*PI/180}" upper="${90*PI/180}" effort="6" velocity="8"/>
-    </joint>
-    <xacro:delta_arm prefix="3"/>
-    <joint name="arm_3_delta_joint" type="revolute">
-        <parent link="base_link"/>
-        <child link="arm_3_link"/>
-        <origin xyz="-0.0555 -0.09612 0.0" rpy="0.0 0.0 ${120*PI/180}"/>
-        <axis xyz="0.0 1 0.0"/>
-        <dynamics damping="0.7"/>
-        <limit lower="${-20*PI/180}" upper="${90*PI/180}" effort="6" velocity="8"/>
-    </joint>
-    <link name="mobile_platform">
-        <visual>
-            <geometry>
-                <cylinder radius="0.035" length="${inch/4}"/>
-            </geometry>
-            <origin xyz="0.0 0.0 0.0" rpy="0.0 0.0 0.0"/>
-            <material name="orange">
-                <color rgba="${255/255} ${108/255} ${10/255} 1.0"/>
-            </material>
-        </visual>
-        <collision>
-            <geometry>
-                <cylinder radius="0.035" length="${inch/4}"/>
-            </geometry>
-            <origin xyz="0.0 0.0 0.0" rpy="0.0 0.0 0.0"/>
-        </collision>
-        <xacro:inertial_cylinder mass="0.1" length="${inch/4}" radius="0.035">
-            <origin xyz="0.0 0.0 0.0" rpy="0.0 0.0 0.0"/>
-        </xacro:inertial_cylinder>
-    </link>
-    <joint name="1_mobile_joint" type="fixed">
-        <parent link="forearm_1_end_link"/>
-        <child link="mobile_platform"/>
-        <origin xyz="-0.035 0 0" rpy="0 0 0"/>
-    </joint>
-    <link name="2_mobile_virtual_link">
-        <inertial>
-        <origin xyz="0 0 0" rpy="0 0 0"/>
-        <mass value="0.001"/>
-        <inertia
-            ixx="0.0001" ixy="0.0" ixz="0.0"
-            iyy="0.0001" iyz="0.0"
-            izz="0.0001"/>
-        </inertial>
-    </link>
-    <joint name="2_mobile_virtual_joint" type="fixed">
-        <parent link="mobile_platform"/>
-        <child link="2_mobile_virtual_link"/>
-        <origin xyz="0.0175 -0.03031 0" rpy="0 0 ${-120*PI/180}"/>
-    </joint>
-    <link name="3_mobile_virtual_link">
-        <inertial>
-        <origin xyz="0 0 0" rpy="0 0 0"/>
-        <mass value="0.001"/>
-        <inertia
-            ixx="0.0001" ixy="0.0" ixz="0.0"
-            iyy="0.0001" iyz="0.0"
-            izz="0.0001"/>
-        </inertial>
-    </link>
-    <joint name="3_mobile_virtual_joint" type="fixed">
-        <parent link="mobile_platform"/>
-        <child link="3_mobile_virtual_link"/>
-        <origin xyz="0.0175 0.03031 0" rpy="0 0 ${120*PI/180}"/>
-    </joint>
-    <gazebo>
-        <joint name="2_end_joint" type="fixed">
-            <parent>forearm_2_end_link</parent>
-            <child>2_mobile_virtual_link</child>
-            <pose> 0 0 0 0 0 0 </pose>
-        </joint>
-        <joint name="left_end_joint" type="fixed">
-            <parent>forearm_3_end_link</parent>
-            <child>3_mobile_virtual_link</child>
-            <pose> 0 0 0 0 0 0 </pose>
-        </joint>
-    </gazebo>
+  </gazebo>
 </robot>

File: urdf/gazebo_stuff.xacro (robot description, xacro)
@@ -2,52 +2,163 @@
 <robot xmlns:xacro="http://www.ros.org/wiki/xacro">
     <physics type='ode'>
-        <max_step_size>0.001</max_step_size>
-        <real_time_factor>0.1</real_time_factor>
-        <real_time_update_rate>1000</real_time_update_rate>
-        <gravity>0 0 -9.8</gravity>
-    </physics>
-    <gazebo>
-        <plugin name="gazebo_ros2_control" filename="libgazebo_ros2_control.so">
-            <robotNamespace></robotNamespace>
-            <robotSimType>gazebo_ros2_control/DefaultRobotHWSim</robotSimType>
-        </plugin>
+    <max_step_size>0.001</max_step_size>
+    <real_time_factor>0.1</real_time_factor>
+    <real_time_update_rate>1000</real_time_update_rate>
+    <gravity>0 0 -9.8</gravity>
+  </physics>
+  <gazebo>
+    <plugin name="gazebo_ros_control" filename="libgazebo_ros_control.so">
+      <robotNamespace></robotNamespace>
+      <robotSimType>gazebo_ros_control/DefaultRobotHWSim</robotSimType>
+      <legacyModeNS>true</legacyModeNS>
+    </plugin>
+  </gazebo>
+  <gazebo reference="base_link">
+    <material>Gazebo/Orange</material>
+    <selfCollide>false</selfCollide>
+  </gazebo>
+  <gazebo reference="end_link">
+    <material>Gazebo/Orange</material>
+    <selfCollide>false</selfCollide>
+  </gazebo>
+  <transmission name="front_delta_arm_joint_trans">
+    <type>transmission_interface/SimpleTransmission</type>
+    <joint name="front_delta_arm_joint">
+      <hardwareInterface>hardware_interface/EffortJointInterface</hardwareInterface>
+    </joint>
+    <actuator name="front_delta_arm_joint_motor">
+      <hardwareInterface>hardware_interface/EffortJointInterface</hardwareInterface>
+      <mechanicalReduction>1</mechanicalReduction>
+    </actuator>
+  </transmission>
+  <transmission name="right_delta_arm_joint_trans">
+    <type>transmission_interface/SimpleTransmission</type>
+    <joint name="right_delta_arm_joint">
+      <hardwareInterface>hardware_interface/EffortJointInterface</hardwareInterface>
+    </joint>
+    <actuator name="right_delta_arm_joint_motor">
+      <hardwareInterface>hardware_interface/EffortJointInterface</hardwareInterface>
+      <mechanicalReduction>1</mechanicalReduction>
+    </actuator>
+  </transmission>
+  <transmission name="left_delta_arm_joint_trans">
+    <type>transmission_interface/SimpleTransmission</type>
+    <joint name="left_delta_arm_joint">
+      <hardwareInterface>hardware_interface/EffortJointInterface</hardwareInterface>
+    </joint>
+    <actuator name="left_delta_arm_joint_motor">
+      <hardwareInterface>hardware_interface/EffortJointInterface</hardwareInterface>
+      <mechanicalReduction>1</mechanicalReduction>
+    </actuator>
+  </transmission>
+  <xacro:macro name="delta_arm_gazebo" params="prefix">
+    <gazebo reference="${prefix}upper_link">
+      <material>Gazebo/Black</material>
+      <selfCollide>false</selfCollide>
     </gazebo>
-    <gazebo reference="base_link">
-        <material>Gazebo/Orange</material>
-        <selfCollide>false</selfCollide>
+    <gazebo reference="${prefix}lower_top_link">
+      <material>Gazebo/Grey</material>
+      <selfCollide>false</selfCollide>
     </gazebo>
-    <gazebo reference="end_link">
-        <material>Gazebo/Orange</material>
-        <selfCollide>false</selfCollide>
+    <gazebo reference="${prefix}lower_right_link">
+      <material>Gazebo/Grey</material>
+      <selfCollide>false</selfCollide>
     </gazebo>
-    <transmission name="arm_1_delta_joint_trans">
-        <type>transmission_interface/Transmission</type>
-        <joint name="arm_1_delta_joint">
-        <hardwareInterface>hardware_interface::EffortJoint</hardwareInterface>
-        </joint>
-            <actuator name="arm_1_delta_joint_motor">
-            <hardwareInterface>hardware_interface::EffortJoint</hardwareInterface>
-            <mechanicalReduction>1</mechanicalReduction>
-        </actuator>
+    <gazebo reference="${prefix}lower_left_link">
+      <material>Gazebo/Grey</material>
+      <selfCollide>false</selfCollide>
+    </gazebo>
+    <gazebo reference="${prefix}lower_bottom_link">
+      <material>Gazebo/Grey</material>
+      <selfCollide>false</selfCollide>
+    </gazebo>
+    <gazebo reference="${prefix}lower_end_link">
+      <material>Gazebo/Black</material>
+      <selfCollide>false</selfCollide>
+    </gazebo>
+    <transmission name="${prefix}upper_joint_trans">
+      <type>transmission_interface/SimpleTransmission</type>
+      <joint name="${prefix}upper_joint">
+        <hardwareInterface>hardware_interface/EffortJointInterface</hardwareInterface>
+      </joint>
+      <actuator name="${prefix}upper_joint_motor">
+        <hardwareInterface>hardware_interface/EffortJointInterface</hardwareInterface>
+        <mechanicalReduction>1</mechanicalReduction>
+      </actuator>
     </transmission>
-    <transmission name="arm_2_delta_joint_trans">
-        <type>transmission_interface/Transmission</type>
-        <joint name="arm_2_delta_joint">
-        <hardwareInterface>hardware_interface::EffortJoint</hardwareInterface>
-        </joint>
-            <actuator name="arm_2_delta_joint_motor">
-            <hardwareInterface>hardware_interface::EffortJoint</hardwareInterface>
-            <mechanicalReduction>1</mechanicalReduction>
-        </actuator>
+    <transmission name="${prefix}lower_top_rignt_joint_trans">
+      <type>transmission_interface/SimpleTransmission</type>
+      <joint name="${prefix}lower_top_rignt_joint">
+        <hardwareInterface>hardware_interface/EffortJointInterface</hardwareInterface>
+      </joint>
+      <actuator name="${prefix}lower_top_rignt_joint_motor">
+        <hardwareInterface>hardware_interface/EffortJointInterface</hardwareInterface>
+        <mechanicalReduction>1</mechanicalReduction>
+      </actuator>
     </transmission>
-    <transmission name="arm_3_delta_joint_trans">
-        <type>transmission_interface/Transmission</type>
-        <joint name="arm_3_delta_joint">
-        <hardwareInterface>hardware_interface::EffortJoint</hardwareInterface>
-        </joint>
-            <actuator name="arm_3_delta_joint_motor">
-            <hardwareInterface>hardware_interface::EffortJoint</hardwareInterface>
-            <mechanicalReduction>1</mechanicalReduction>
-        </actuator>
+    <transmission name="${prefix}lower_top_left_joint_trans">
+      <type>transmission_interface/SimpleTransmission</type>
+      <joint name="${prefix}lower_top_left_joint">
+        <hardwareInterface>hardware_interface/EffortJointInterface</hardwareInterface>
+      </joint>
+      <actuator name="${prefix}lower_top_left_joint_motor">
+        <hardwareInterface>hardware_interface/EffortJointInterface</hardwareInterface>
+        <mechanicalReduction>1</mechanicalReduction>
+      </actuator>
     </transmission>
+    <transmission name="${prefix}lower_right_bottom_joint_trans">
+      <type>transmission_interface/SimpleTransmission</type>
+      <joint name="${prefix}lower_right_bottom_joint">
+        <hardwareInterface>hardware_interface/EffortJointInterface</hardwareInterface>
+      </joint>
+      <actuator name="${prefix}lower_right_bottom_joint_motor">
+        <hardwareInterface>hardware_interface/EffortJointInterface</hardwareInterface>
+        <mechanicalReduction>1</mechanicalReduction>
+      </actuator>
+    </transmission>
+    <transmission name="${prefix}lower_bottom_end_joint_trans">
+      <type>transmission_interface/SimpleTransmission</type>
+      <joint name="${prefix}lower_bottom_end_joint">
+        <hardwareInterface>hardware_interface/EffortJointInterface</hardwareInterface>
+      </joint>
+      <actuator name="${prefix}lower_bottom_end_joint_motor">
+        <hardwareInterface>hardware_interface/EffortJointInterface</hardwareInterface>
+        <mechanicalReduction>1</mechanicalReduction>
+      </actuator>
+    </transmission>
+    <transmission name="${prefix}lower_bottom_virtual_joint_trans">
+      <type>transmission_interface/SimpleTransmission</type>
+      <joint name="${prefix}lower_bottom_virtual_joint">
+        <hardwareInterface>hardware_interface/EffortJointInterface</hardwareInterface>
+      </joint>
+      <actuator name="${prefix}lower_bottom_virtual_joint_motor">
+        <hardwareInterface>hardware_interface/EffortJointInterface</hardwareInterface>
+        <mechanicalReduction>1</mechanicalReduction>
+      </actuator>
+    </transmission>
+  </xacro:macro>
+  <material name="black">
+    <color rgba="0.0 0.0 0.0 1.0"/>
+  </material>
+  <material name="blue">
+    <color rgba="0.0 0.0 0.8 1.0"/>
+  </material>
+  <material name="green">
+    <color rgba="0.0 0.8 0.0 1.0"/>
+  </material>
+  <material name="grey">
+    <color rgba="0.2 0.2 0.2 1.0"/>
+  </material>
+  <material name="orange">
+    <color rgba="${255/255} ${108/255} ${10/255} 1.0"/>
+  </material>
+  <material name="brown">
+    <color rgba="${222/255} ${207/255} ${195/255} 1.0"/>
+  </material>
+  <material name="red">
+    <color rgba="0.8 0.0 0.0 1.0"/>
+  </material>
+  <material name="white">
+    <color rgba="1.0 1.0 1.0 1.0"/>
+  </material>
 </robot>
